File: PCB/ESC/MerlynESC.kicad_pcb (KiCad board)
At the start: 4 copper layers, 30.5 x 31.9 mm, 155 parts, among them M1 BLDC Motor, M2 BLDC Motor, M3 BLDC Motor, M4 BLDC Motor, Q1 JMSL0302AU, Q10 JMSL0302AU, Q11 JMSL0302AU, Q12 JMSL0302AU, Q13 JMSL0302AU, Q14 JMSL0302AU, Q15 JMSL0302AU, Q16 JMSL0302AU, Q17 JMSL0302AU, Q18 JMSL0302AU, Q19 JMSL0302AU, Q2 JMSL0302AU, Q20 JMSL0302AU, Q21 JMSL0302AU, Q22 JMSL0302AU, Q23 JMSL0302AU, Q24 JMSL0302AU, Q3 JMSL0302AU, Q4 JMSL0302AU, Q5 JMSL0302AU, Q6 JMSL0302AU, Q7 JMSL0302AU, Q8 JMSL0302AU, Q9 JMSL0302AU, U1 HT75C0-1, U10 EG6288, U11 EFM8BB21F16G, U2 HT7533-1, U3 EFM8BB21F16G, U4 EG6288, U5 EG6288, U6 EFM8BB21F16G, U7 INA139NA, U8 EG6288, U9 EFM8BB21F16G

Commit message: checkpoint
Parts:
- C11, C12, C13, C17, C18, C19, C3, C8, D1, D2, D3, D4, D5, D6, R11, R13, R15, R21, R26, R31: moved to B.Cu
- moved Q2 79.0 mm to (163.0, 115.6), turned to -90 degrees
- moved Q8 77.2 mm to (165.9, 100.0), turned to -90 degrees
- moved Q4 70.1 mm to (165.9, 107.9), turned to -90 degrees
- moved Q10 67.9 mm to (165.9, 96.0), turned to -90 degrees
- moved R11 64.5 mm to (161.5, 107.5), turned to 180 degrees
- moved R13 62.4 mm to (161.5, 104.9), turned to 180 degrees
- moved R21 62.0 mm to (161.5, 99.7), turned to 180 degrees
- moved R15 61.6 mm to (161.5, 102.3), turned to 180 degrees
- moved Q6 60.7 mm to (165.9, 103.9), turned to -90 degrees
- moved R31 59.6 mm to (161.5, 94.4), turned to 180 degrees
- moved R26 58.5 mm to (161.5, 97.1), turned to 180 degrees
- moved Q12 54.9 mm to (163.0, 88.3), turned to -90 degrees
- moved Q22 53.8 mm to (144.9, 96.0), turned to 90 degrees
- moved Q24 46.1 mm to (144.9, 100.0), turned to 90 degrees
- moved C8 44.6 mm to (160.5, 111.7), turned to 90 degrees
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Routing:
- net +BATT: track 5.97 -> 49.5 mm
- net Net-(D10-K): track 0.00 -> 6.58 mm
- net Net-(D7-K): track 0.00 -> 6.08 mm
- net M3_HIN2: track 0.00 -> 4.63 mm, vias 0 -> 1
- net Net-(D11-K): track 0.00 -> 4.57 mm
- net GND: track 1.61 -> 6.06 mm
- net Net-(D8-K): track 0.00 -> 4.20 mm
- net Net-(D9-K): track 0.00 -> 4.19 mm
- net Net-(D12-K): track 0.00 -> 4.17 mm
- net M4_H01: track 0.00 -> 3.41 mm
- net M3_LIN1: track 0.00 -> 3.28 mm, vias 0 -> 1
- net Net-(D1-K): track 0.00 -> 3.23 mm
- net Net-(D4-K): track 0.00 -> 3.18 mm
- net M3_H01: track 0.00 -> 3.05 mm
- net Net-(U8-VS3): track 0.00 -> 3.03 mm
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
Commit message: checkpoint
Parts:
- C9: moved to B.Cu
- moved R23 64.0 mm to (162.4, 95.3), turned to 90 degrees
- moved R9 63.3 mm to (162.8, 105.0), turned to 90 degrees
- moved R8 63.2 mm to (162.8, 103.3), turned to 90 degrees
- moved R7 62.5 mm to (162.8, 106.7), turned to 90 degrees
- moved R6 61.7 mm to (162.0, 105.0), turned to 90 degrees
- moved R5 61.7 mm to (162.0, 103.3), turned to 90 degrees
- moved R4 61.5 mm to (162.0, 106.7), turned to 90 degrees
- moved R20 61.4 mm to (162.4, 97.0), turned to 90 degrees
- moved R1 60.9 mm to (161.2, 105.0), turned to 90 degrees
- moved R2 60.9 mm to (161.2, 106.7), turned to 90 degrees
- moved R3 60.7 mm to (161.2, 103.3), turned to 90 degrees
- moved R19 60.5 mm to (162.4, 98.7), turned to 90 degrees
- moved R18 60.0 mm to (161.6, 95.3), turned to 90 degrees
- moved R10 58.0 mm to (156.6, 103.2), turned to 180 degrees
- moved R30 57.3 mm to (161.7, 97.0), turned to 90 degrees
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Routing:
- net +BATT: track 49.5 -> 71.2 mm, vias 0 -> 22
- net GND: track 6.06 -> 27.8 mm, vias 0 -> 16
- net +3.3V: track 0.00 -> 6.34 mm
- net Net-(D6-K): track 0.00 -> 4.03 mm
- net M4_HIN3: track 0.00 -> 2.85 mm, vias 0 -> 1
- net M1_LIN1: track 0.00 -> 2.81 mm, vias 0 -> 1
- net M2_LIN1: track 0.00 -> 2.81 mm, vias 0 -> 1
- net M4_LIN1: track 0.00 -> 2.81 mm, vias 0 -> 1
- net M3_HIN2: track 4.63 -> 1.87 mm
- net M2_HIN3: track 0.00 -> 2.63 mm, vias 0 -> 1
- net Net-(U5-VS3): track 0.00 -> 2.62 mm
- net M1_HIN3: track 0.00 -> 2.61 mm, vias 0 -> 1
- net M3_HIN3: track 0.00 -> 2.60 mm, vias 0 -> 1
- net M4_LIN2: track 0.00 -> 2.32 mm, vias 0 -> 1
- net M2_LIN2: track 0.00 -> 2.32 mm, vias 0 -> 1
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- added copper zone on B.Cu, net +BATT
- added copper zone on F.Cu, net +BATT
- added copper zone on B.Cu, net Net-(BT1-+)
Other:
- outline, holes or cut-outs redrawn

Commit message: checkpoint
Parts:
- moved R1 41.2 mm to (120.2, 109.0)
- moved R6 41.2 mm to (121.0, 109.0)
- moved R9 41.2 mm to (121.8, 109.0)
- moved R18 41.2 mm to (120.6, 99.3)
- moved R19 41.2 mm to (121.4, 102.7)
- moved R2 41.2 mm to (120.2, 110.8)
- moved R23 41.2 mm to (121.4, 99.3)
- moved R24 41.2 mm to (119.8, 102.7)
- moved R28 41.2 mm to (119.8, 99.3)
- moved R29 41.2 mm to (120.6, 102.7)
- moved R36 41.2 mm to (109.3, 107.2)
- moved R38 41.2 mm to (108.5, 108.8)
- moved R4 41.2 mm to (121.0, 110.8)
- moved R41 41.2 mm to (108.5, 107.2)
- moved R42 41.2 mm to (109.3, 110.5)
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Routing:
- net +BATT: vias 22 -> 34

Commit message: checkpoint
Parts:
- moved R64 42.8 mm to (150.1, 94.6)
- moved R62 42.6 mm to (150.1, 99.5)
- moved R53 41.5 mm to (148.6, 97.1), turned to 90 degrees
- moved R58 41.5 mm to (150.1, 97.1), turned to 90 degrees
- moved R63 41.5 mm to (149.3, 97.1), turned to 90 degrees
- moved R38 41.4 mm to (149.3, 102.0)
- moved R43 41.4 mm to (150.1, 102.0)
- moved R48 41.4 mm to (148.6, 102.0)
- moved R59 41.2 mm to (149.3, 94.6)
- moved R1 41.2 mm to (161.2, 105.0)
- moved R6 41.2 mm to (162.0, 105.0)
- moved R9 41.2 mm to (162.8, 105.0)
- moved R18 41.2 mm to (161.6, 95.3)
- moved R19 41.2 mm to (162.4, 98.7)
- moved R2 41.2 mm to (161.2, 106.7)
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Connections:
- U11 pad 1: M4_BEMF3 -> M4_BEMF1
- U11 pad 19: M4_BEMFCommon -> M4_BEMF3
- U11 pad 2: M4_BEMF2 -> M4_BEMFCommon
- U11 pad 20: M4_BEMF1 -> M4_BEMF2
Routing:
- net +BATT: track 71.2 -> 3.40 mm, vias 34 -> 22
- net GND: track 27.8 -> 13.5 mm
- net M4_PHASE3: track 0.00 -> 13.3 mm, vias 0 -> 1
- net M4_PHASE2: track 0.00 -> 10.1 mm, vias 0 -> 1
- net M4_PHASE1: track 0.00 -> 7.98 mm, vias 0 -> 1
- net M4_BEMFCommon: track 0.00 -> 4.37 mm
- net Net-(Q19-G): track 0.00 -> 0.67 mm, vias 0 -> 1
- added copper zone on F.Cu, net GND
- added copper zone on B.Cu, net M1_PHASE1
- added copper zone on F.Cu, net M1_PHASE1
- added copper zone on B.Cu, net M1_PHASE2
- added copper zone on F.Cu, net M1_PHASE2
- added copper zone on B.Cu, net M1_PHASE3
- added copper zone on F.Cu, net M1_PHASE3
- added copper zone on B.Cu, net M2_PHASE1
- added copper zone on F.Cu, net M2_PHASE1
- added copper zone on B.Cu, net M2_PHASE2
- added copper zone on F.Cu, net M2_PHASE2
- added copper zone on B.Cu, net M2_PHASE3
- added copper zone on F.Cu, net M2_PHASE3
- added copper zone on B.Cu, net M3_PHASE1
- added copper zone on F.Cu, net M3_PHASE1
- added copper zone on B.Cu, net M3_PHASE2
- added copper zone on F.Cu, net M3_PHASE2
- added copper zone on B.Cu, net M3_PHASE3
- added copper zone on F.Cu, net M3_PHASE3
- added copper zone on B.Cu, net M4_PHASE1
- added copper zone on F.Cu, net M4_PHASE1
- added copper zone on B.Cu, net M4_PHASE2
- added copper zone on F.Cu, net M4_PHASE2
- added copper zone on B.Cu, net M4_PHASE3
- added copper zone on F.Cu, net M4_PHASE3
Other:
- copper layers 4 -> 6

Commit message: checkpoint
Parts:
- moved R7 5.29 mm to (160.6, 101.9), turned to -90 degrees
- moved R2 4.96 mm to (162.4, 101.9), turned to -90 degrees
- moved R4 4.86 mm to (161.5, 101.9), turned to -90 degrees
- moved R36 2.97 mm to (148.5, 106.9)
- moved R46 2.97 mm to (150.2, 106.9)
- moved R47 2.97 mm to (150.2, 104.5)
- moved R9 2.82 mm to (160.6, 106.8), turned to -90 degrees
- moved R30 2.61 mm to (160.6, 99.4), turned to -90 degrees
- moved R37 2.61 mm to (148.5, 104.5)
- moved R42 2.58 mm to (149.3, 104.5)
- moved R25 2.48 mm to (161.5, 99.4), turned to -90 degrees
- moved R41 2.46 mm to (149.3, 106.9)
- moved R20 2.40 mm to (162.4, 99.4), turned to -90 degrees
- moved R8 2.39 mm to (160.6, 104.3), turned to -90 degrees
- moved R1 2.16 mm to (162.4, 106.8), turned to -90 degrees
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Connections:
- U3 pad 1: M1_BEMF3 -> M1_BEMF1
- U3 pad 19: M1_BEMFCommon -> M1_BEMF3
- U3 pad 2: M1_BEMF2 -> M1_BEMFCommon
- U3 pad 20: M1_BEMF1 -> M1_BEMF2
- U6 pad 1: M2_BEMF3 -> M2_BEMF1
- U6 pad 19: M2_BEMFCommon -> M2_BEMF3
- U6 pad 2: M2_BEMF2 -> M2_BEMFCommon
- U6 pad 20: M2_BEMF1 -> M2_BEMF2
- U9 pad 1: M3_BEMF3 -> M3_BEMF1
- U9 pad 19: M3_BEMFCommon -> M3_BEMF3
- U9 pad 2: M3_BEMF2 -> M3_BEMFCommon
- U9 pad 20: M3_BEMF1 -> M3_BEMF2
Routing:
- net Net-(Q20-G): track 0.00 -> 17.0 mm, vias 0 -> 2
- net Net-(Q22-G): track 0.00 -> 13.3 mm, vias 0 -> 2
- net Net-(Q24-G): track 0.00 -> 11.9 mm, vias 0 -> 2
- net M2_BEMF1: track 0.00 -> 11.1 mm
- net Net-(Q1-G): track 0.00 -> 10.9 mm, vias 0 -> 2
- net M1_BEMF1: track 0.00 -> 10.3 mm
- net Net-(Q19-G): track 0.67 -> 11.0 mm, vias 1 -> 2
- net M2_BEMF2: track 0.00 -> 10.0 mm
- net M1_BEMF2: track 0.00 -> 9.26 mm
- net M3_BEMF1: track 0.00 -> 8.82 mm
- net M4_BEMF1: track 0.00 -> 8.48 mm
- net Net-(Q11-G): track 0.00 -> 7.83 mm, vias 0 -> 2
- net Net-(Q17-G): track 0.00 -> 7.82 mm, vias 0 -> 2
- net Net-(Q3-G): track 0.00 -> 7.72 mm, vias 0 -> 2
- net Net-(Q21-G): track 0.00 -> 7.72 mm, vias 0 -> 2
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- added copper zone on In3.Cu, net +BATT
- added copper zone on In4.Cu, net +BATT
- added copper zone on In1.Cu, net GND
- added copper zone on In2.Cu, net GND
- added copper zone on In1.Cu, net M1_PHASE1
- added copper zone on In2.Cu, net M1_PHASE1
- added copper zone on In3.Cu, net M1_PHASE1
- added copper zone on In4.Cu, net M1_PHASE1
- added copper zone on In1.Cu, net M1_PHASE2
- added copper zone on In2.Cu, net M1_PHASE2
- added copper zone on In3.Cu, net M1_PHASE2
- added copper zone on In4.Cu, net M1_PHASE2
- added copper zone on In1.Cu, net M1_PHASE3
- added copper zone on In2.Cu, net M1_PHASE3
- added copper zone on In3.Cu, net M1_PHASE3
- added copper zone on In4.Cu, net M1_PHASE3
- added copper zone on In1.Cu, net M2_PHASE1
- added copper zone on In2.Cu, net M2_PHASE1
- added copper zone on In3.Cu, net M2_PHASE1
- added copper zone on In4.Cu, net M2_PHASE1
- added copper zone on In1.Cu, net M2_PHASE2
- added copper zone on In2.Cu, net M2_PHASE2
- added copper zone on In3.Cu, net M2_PHASE2
- added copper zone on In4.Cu, net M2_PHASE2
- added copper zone on In1.Cu, net M2_PHASE3
- added copper zone on In2.Cu, net M2_PHASE3
- added copper zone on In3.Cu, net M2_PHASE3
- added copper zone on In4.Cu, net M2_PHASE3
- added copper zone on In1.Cu, net M3_PHASE1
- added copper zone on In2.Cu, net M3_PHASE1
- added copper zone on In3.Cu, net M3_PHASE1
- added copper zone on In4.Cu, net M3_PHASE1
- added copper zone on In1.Cu, net M3_PHASE2
- added copper zone on In2.Cu, net M3_PHASE2
- added copper zone on In3.Cu, net M3_PHASE2
- added copper zone on In4.Cu, net M3_PHASE2
- added copper zone on In1.Cu, net M3_PHASE3
- added copper zone on In2.Cu, net M3_PHASE3
- added copper zone on In3.Cu, net M3_PHASE3
- added copper zone on In4.Cu, net M3_PHASE3
- added copper zone on In1.Cu, net M4_PHASE1
- added copper zone on In2.Cu, net M4_PHASE1
- added copper zone on In3.Cu, net M4_PHASE1
- added copper zone on In4.Cu, net M4_PHASE1
- added copper zone on In1.Cu, net M4_PHASE2
- added copper zone on In2.Cu, net M4_PHASE2
- added copper zone on In3.Cu, net M4_PHASE2
- added copper zone on In4.Cu, net M4_PHASE2
- added copper zone on In1.Cu, net M4_PHASE3
- added copper zone on In2.Cu, net M4_PHASE3
- added copper zone on In3.Cu, net M4_PHASE3
- added copper zone on In4.Cu, net M4_PHASE3
- added copper zone on In3.Cu, net Net-(BT1-+)
- added copper zone on In4.Cu, net Net-(BT1-+)
- removed copper zone on F.Cu, net +BATT

Commit message: checkpoint
Parts:
- moved C21 4.74 mm to (157.8, 108.4)
- moved R35 0.38 mm to (154.9, 93.4), turned to 180 degrees
Routing:
- net M3_DSHOT: track 0.00 -> 23.1 mm, vias 0 -> 2
- net M1_DSHOT: track 0.00 -> 22.8 mm, vias 0 -> 2
- net Net-(Q2-G): track 0.00 -> 18.2 mm, vias 0 -> 2
- net M4_DSHOT: track 0.00 -> 18.0 mm, vias 0 -> 2
- net M2_DSHOT: track 0.00 -> 15.4 mm, vias 0 -> 2
- net M3_PHASE3: track 2.01 -> 17.2 mm, vias 0 -> 1
- net M2_PHASE3: track 0.00 -> 14.8 mm, vias 0 -> 1
- net Net-(Q4-G): track 0.00 -> 12.7 mm, vias 0 -> 2
- net Net-(Q8-G): track 0.00 -> 10.9 mm, vias 0 -> 2
- net Net-(Q6-G): track 0.00 -> 10.7 mm, vias 0 -> 2
- net Net-(Q14-G): track 0.66 -> 10.8 mm, vias 1 -> 2
- net Net-(Q18-G): track 0.00 -> 9.95 mm, vias 0 -> 2
- net Net-(Q10-G): track 0.00 -> 8.36 mm, vias 0 -> 2
- net M1_PHASE2: track 0.00 -> 8.05 mm, vias 0 -> 1
- net Net-(Q12-G): track 0.00 -> 7.64 mm, vias 0 -> 2
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
Commit message: checkpoint
Routing:
- net +3.3V: track 6.34 -> 43.1 mm, vias 0 -> 5
- net Net-(U7-OUT): track 1.02 -> 20.0 mm, vias 2 -> 3
- net M2_PHASE1: track 3.57 -> 7.31 mm, vias 1 -> 7
- net M3_PHASE1: track 6.13 -> 9.67 mm, vias 1 -> 7
- net M1_PHASE3: track 7.54 -> 11.0 mm, vias 1 -> 7
- net M4_PHASE3: track 7.36 -> 10.8 mm, vias 1 -> 7
- net Net-(Q11-G): track 7.83 -> 9.98 mm
- net M1_PHASE1: track 7.25 -> 9.38 mm, vias 1 -> 13
- net M2_PHASE2: track 4.55 -> 5.87 mm, vias 1 -> 7
- net M3_PHASE2: track 6.74 -> 8.00 mm, vias 1 -> 7
- net Net-(Q3-G): track 7.72 -> 8.79 mm
- net M1_PHASE2: track 8.05 -> 9.08 mm, vias 1 -> 7
- net GND: track 14.9 -> 15.7 mm, vias 43 -> 42
- net M4_PHASE2: track 6.63 -> 7.44 mm, vias 1 -> 7
- net Net-(Q4-G): track 12.7 -> 13.5 mm
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- removed copper zone on In1.Cu, net M1_PHASE1
- removed copper zone on In2.Cu, net M1_PHASE1
- removed copper zone on In3.Cu, net M1_PHASE1
- removed copper zone on In4.Cu, net M1_PHASE1
- removed copper zone on In1.Cu, net M1_PHASE2
- removed copper zone on In2.Cu, net M1_PHASE2
- removed copper zone on In3.Cu, net M1_PHASE2
- removed copper zone on In4.Cu, net M1_PHASE2
- removed copper zone on In1.Cu, net M1_PHASE3
- removed copper zone on In2.Cu, net M1_PHASE3
- removed copper zone on In3.Cu, net M1_PHASE3
- removed copper zone on In4.Cu, net M1_PHASE3
- removed copper zone on In1.Cu, net M2_PHASE1
- removed copper zone on In2.Cu, net M2_PHASE1
- removed copper zone on In3.Cu, net M2_PHASE1
- removed copper zone on In4.Cu, net M2_PHASE1
- removed copper zone on In1.Cu, net M2_PHASE2
- removed copper zone on In2.Cu, net M2_PHASE2
- removed copper zone on In3.Cu, net M2_PHASE2
- removed copper zone on In4.Cu, net M2_PHASE2
- removed copper zone on In1.Cu, net M2_PHASE3
- removed copper zone on In2.Cu, net M2_PHASE3
- removed copper zone on In3.Cu, net M2_PHASE3
- removed copper zone on In4.Cu, net M2_PHASE3
- removed copper zone on In1.Cu, net M3_PHASE1
- removed copper zone on In2.Cu, net M3_PHASE1
- removed copper zone on In3.Cu, net M3_PHASE1
- removed copper zone on In4.Cu, net M3_PHASE1
- removed copper zone on In1.Cu, net M3_PHASE2
- removed copper zone on In2.Cu, net M3_PHASE2
- removed copper zone on In3.Cu, net M3_PHASE2
- removed copper zone on In4.Cu, net M3_PHASE2
- removed copper zone on In1.Cu, net M3_PHASE3
- removed copper zone on In2.Cu, net M3_PHASE3
- removed copper zone on In3.Cu, net M3_PHASE3
- removed copper zone on In4.Cu, net M3_PHASE3
- removed copper zone on In1.Cu, net M4_PHASE1
- removed copper zone on In2.Cu, net M4_PHASE1
- removed copper zone on In3.Cu, net M4_PHASE1
- removed copper zone on In4.Cu, net M4_PHASE1
- removed copper zone on In1.Cu, net M4_PHASE2
- removed copper zone on In2.Cu, net M4_PHASE2
- removed copper zone on In3.Cu, net M4_PHASE2
- removed copper zone on In4.Cu, net M4_PHASE2
- removed copper zone on In1.Cu, net M4_PHASE3
- removed copper zone on In2.Cu, net M4_PHASE3
- removed copper zone on In3.Cu, net M4_PHASE3
- removed copper zone on In4.Cu, net M4_PHASE3

Commit message: checkpoint
Routing:
- net +12V: track 13.8 -> 110.8 mm, vias 0 -> 11
- net GND: track 15.7 -> 27.6 mm, vias 42 -> 56
- net Net-(BT1-+): track 1.99 -> 5.70 mm
- net M4_PHASE1: track 6.96 -> 8.36 mm
- net M1_LIN2: track 1.02 -> 2.30 mm
- net M2_PHASE3: track 14.8 -> 16.0 mm
- net M1_LIN3: track 1.06 -> 1.97 mm
- net Net-(Q20-G): track 17.0 -> 17.8 mm
- net M3_PHASE1: track 9.67 -> 10.4 mm
- net Net-(Q2-G): track 18.2 -> 18.9 mm
- net Net-(Q21-G): track 8.44 -> 9.08 mm
- net Net-(Q10-G): track 8.36 -> 8.91 mm
