File: PCB/ESC/MerlynESC.kicad_sch (KiCad schematic)
At the start: 45 parts, among them M1 BLDC Motor, Q1 JMSL0302AU, Q2 JMSL0302AU, Q3 JMSL0302AU, Q4 JMSL0302AU, Q5 JMSL0302AU, Q6 JMSL0302AU, U1 HT75C0-1, U2 HT7533-1, U3 EFM8BB21F16G, U4 EG6288

Commit message: minor esc fixes
Parts:
- R11, R12, R13, R14, R15, R16: value 22 -> 10; LCSC Part C25092 -> C25077
Connections:
- net +12V: now also U1.3 (VOUT)
- net GND: now also C2.1
Other:
- moved on the sheet: C2
Changed lines of the file:
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@@
 		(color 0 0 0 0)
 	)
+	(junction
+		(at 124.46 64.77)
+		(diameter 0)
+		(color 0 0 0 0)
+	)
 	(no_connect
 		(at 292.1 146.05)
@@
 	(wire
 		(pts
-			(xy 121.92 64.77) (xy 124.46 64.77)
-		)
-		(stroke
-			(width 0)
-			(type default)
-		)
-	)
-	(wire
-		(pts
 			(xy 240.03 128.27) (xy 240.03 130.81)
 		)
@@
 	(wire
 		(pts
-			(xy 121.92 66.04) (xy 121.92 64.77)
-		)
-		(stroke
-			(width 0)
-			(type default)
-		)
-	)
-	(wire
-		(pts
 			(xy 199.39 62.23) (xy 199.39 54.61)
 		)
@@
 	(wire
 		(pts
+			(xy 121.92 64.77) (xy 121.92 71.12)
+		)
+		(stroke
+			(width 0)
+			(type default)
+		)
+	)
+	(wire
+		(pts
 			(xy 107.95 64.77) (xy 119.38 64.77)
 		)
@@
 	(wire
 		(pts
+			(xy 127 64.77) (xy 124.46 64.77)
+		)
+		(stroke
+			(width 0)
+			(type default)
+		)
+	)
+	(wire
+		(pts
 			(xy 107.95 71.12) (xy 107.95 69.85)
 		)
@@
 	(wire
 		(pts
-			(xy 314.96 111.76) (xy 320.04 111.76)
+			(xy 314.96 111.76) (xy 321.31 111.76)
 		)
 		(stroke
@@
 	(wire
 		(pts
+			(xy 121.92 64.77) (xy 124.46 64.77)
+		)
+		(stroke
+			(width 0)
+			(type default)
+		)
+	)
+	(wire
+		(pts
 			(xy 204.47 69.85) (xy 207.01 69.85)
 		)
@@
 			)
 		)
-		(property "Value" "22"
+		(property "Value" "10"
 			(at 216.916 71.12 90)
 			(effects
@@
 			)
 		)
-		(property "Datasheet" "0402, 22r"
+		(property "Datasheet" "0402, 10r"
 			(at 215.9 71.12 0)
 			(effects
@@
 			)
 		)
-		(property "LCSC Part" "C25092"
+		(property "LCSC Part" "C25077"
 			(at 215.9 71.12 0)
 			(effects
@@
 	(symbol
 		(lib_id "Device:C_Small")
-		(at 121.92 68.58 0)
+		(at 127 67.31 0)
 		(mirror x)
 		(unit 1)
@@
 		(dnp no)
 		(property "Reference" "C2"
-			(at 127.254 68.58 0)
+			(at 132.334 67.31 0)
 			(effects
 				(font
@@
 		)
 		(property "Value" "10uF"
-			(at 127.254 70.358 0)
+			(at 132.334 69.088 0)
 			(effects
 				(font
@@
 		)
 		(property "Footprint" "Capacitor_SMD:C_0603_1608Metric"
-			(at 121.92 68.58 0)
+			(at 127 67.31 0)
 			(effects
 				(font
@@
 		)
 		(property "Datasheet" "0603, 10uF, 25v"
-			(at 121.92 68.58 0)
+			(at 127 67.31 0)
 			(effects
 				(font
@@
 		)
 		(property "Description" "Unpolarized capacitor, small symbol"
-			(at 121.92 68.58 0)
+			(at 127 67.31 0)
 			(effects
 				(font
@@
 		)
 		(property "LCSC Part" "C96446"
-			(at 121.92 68.58 0)
+			(at 127 67.31 0)
 			(effects
 				(font
@@
 			)
 		)
-		(property "Value" "22"
+		(property "Value" "10"
 			(at 216.916 96.52 90)
 			(effects
@@
 			)
 		)
-		(property "Datasheet" "0402, 22r"
+		(property "Datasheet" "0402, 10r"
 			(at 215.9 96.52 0)
 			(effects
@@
 			)
 		)
-		(property "LCSC Part" "C25092"
+		(property "LCSC Part" "C25077"
 			(at 215.9 96.52 0)
 			(effects
@@
 			)
 		)
-		(property "Value" "22"
+		(property "Value" "10"
 			(at 257.556 71.12 90)
 			(effects
@@
 			)
 		)
-		(property "Datasheet" "0402, 22r"
+		(property "Datasheet" "0402, 10r"
 			(at 256.54 71.12 0)
 			(effects
@@
 			)
 		)
-		(property "LCSC Part" "C25092"
+		(property "LCSC Part" "C25077"
 			(at 256.54 71.12 0)
 			(effects
@@
 			)
 		)
-		(property "Value" "22"
+		(property "Value" "10"
 			(at 176.276 96.52 90)
 			(effects
@@
 			)
 		)
-		(property "Datasheet" "0402, 22r"
+		(property "Datasheet" "0402, 10r"
 			(at 175.26 96.52 0)
 			(effects
@@
 			)
 		)
-		(property "LCSC Part" "C25092"
+		(property "LCSC Part" "C25077"
 			(at 175.26 96.52 0)
 			(effects
@@
 	(symbol
 		(lib_id "power:GND")
-		(at 320.04 111.76 180)
+		(at 321.31 111.76 0)
+		(mirror y)
 		(unit 1)
 		(exclude_from_sim no)
@@
 		(dnp no)
 		(property "Reference" "#PWR013"
-			(at 320.04 105.41 0)
+			(at 321.31 118.11 0)
 			(effects
 				(font
@@
 		)
 		(property "Value" "GND"
-			(at 320.04 108.204 0)
+			(at 321.31 115.316 0)
 			(effects
 				(font
@@
 		)
 		(property "Footprint" ""
-			(at 320.04 111.76 0)
+			(at 321.31 111.76 0)
 			(effects
 				(font
@@
 		)
 		(property "Datasheet" ""
-			(at 320.04 111.76 0)
+			(at 321.31 111.76 0)
 			(effects
 				(font
@@
 		)
 		(property "Description" "Power symbol creates a global label with name \"GND\" , ground"
-			(at 320.04 111.76 0)
+			(at 321.31 111.76 0)
 			(effects
 				(font
@@
 			)
 		)
-		(property "Value" "22"
+		(property "Value" "10"
 			(at 257.556 96.52 90)
 			(effects
@@
 			)
 		)
-		(property "Datasheet" "0402, 22r"
+		(property "Datasheet" "0402, 10r"
 			(at 256.54 96.52 0)
 			(effects
@@
 			)
 		)
-		(property "LCSC Part" "C25092"
+		(property "LCSC Part" "C25077"
 			(at 256.54 96.52 0)
 			(effects
@@
 		)
 		(property "Value" "+BATT"
-			(at 118.618 59.944 0)
+			(at 117.602 59.944 0)
 			(effects
 				(font
@@
 	)
 	(symbol
+		(lib_id "power:GND")
+		(at 127 69.85 0)
+		(unit 1)
+		(exclude_from_sim no)
+		(in_bom yes)
+		(on_board yes)
+		(dnp no)
+		(property "Reference" "#PWR026"
+			(at 127 76.2 0)
+			(effects
+				(font
+					(size 1.27 1.27)
+				)
+				(hide yes)
+			)
+		)
+		(property "Value" "GND"
+			(at 127 73.406 0)
+			(effects
+				(font
+					(size 1.27 1.27)
+				)
+			)
+		)
+		(property "Footprint" ""
+			(at 127 69.85 0)
+			(effects
+				(font
+					(size 1.27 1.27)
+				)
+				(hide yes)
+			)
+		)
+		(property "Datasheet" ""
+			(at 127 69.85 0)
+			(effects
+				(font
+					(size 1.27 1.27)
+				)
+				(hide yes)
+			)
+		)
+		(property "Description" "Power symbol creates a global label with name \"GND\" , ground"
+			(at 127 69.85 0)
+			(effects
+				(font
+					(size 1.27 1.27)
+				)
+				(hide yes)
+			)
+		)
+		(pin "1"
+		)
+		(instances
+			(project "MerlynESC"
+				(path "/c59754d8-0226-4494-a77d-f4c2074bdb76"
+					(reference "#PWR026")
+					(unit 1)
+				)
+			)
+		)
+	)
+	(symbol
 		(lib_id "Device:R_Small")
 		(at 205.74 125.73 0)
@@
 		(lib_id "power:+BATT")
 		(at 124.46 63.5 0)
+		(mirror y)
 		(unit 1)
 		(exclude_from_sim no)
@@
 		)
 		(property "Value" "+12V"
-			(at 124.968 59.944 0)
+			(at 125.476 59.944 0)
 			(effects
 				(font
@@
 			)
 		)
-		(property "Value" "22"
+		(property "Value" "10"
 			(at 176.276 71.12 90)
 			(effects
@@
 			)
 		)
-		(property "Datasheet" "0402, 22r"
+		(property "Datasheet" "0402, 10r"
 			(at 175.26 71.12 0)
 			(effects
@@
 			)
 		)
-		(property "LCSC Part" "C25092"
+		(property "LCSC Part" "C25077"
 			(at 175.26 71.12 0)
 			(effects

Commit message: checkpoint
Parts:
- added C15, C16, C20, C21: 0.1uF, Capacitor_SMD:C_0402_1005Metric, symbol Device:C_Small
- added C17, C18, C19: 1uF, Capacitor_SMD:C_0402_1005Metric, symbol Device:C_Small
- added D4, D5, D6: T4, Diode_SMD:D_SOD-923, symbol Device:D_Small
- added M2: BLDC Motor, symbol MerlynESC:BLDC Motor
- added Q10, Q11, Q12, Q7, Q8, Q9: JMSL0302AU, easyeda2kicad:DFN-8_L3.2-W3.1-P0.65-LS3.4-BL, symbol MerlynESC:JMSL0302AU
- added R17: HOYLR2512E, easyeda2kicad:R2512, symbol MerlynESC:HOYLR2512E-3W-0.5MR-1%
- added R18, R23, R28: 4.7k, Resistor_SMD:R_0402_1005Metric, symbol Device:R_Small
- added R19, R24, R29, R33: 1k, Resistor_SMD:R_0402_1005Metric, symbol Device:R_Small
- added R20, R25, R30: 10k, Resistor_SMD:R_0402_1005Metric, symbol Device:R_Small
- added R21, R22, R26, R27, R31, R32: 10, Resistor_SMD:R_0402_1005Metric, symbol Device:R_Small
- added R34, R35: 39k, Resistor_SMD:R_0402_1005Metric, symbol Device:R_Small
- added U5: EG6288, easyeda2kicad:QFN-24_L4.0-W4.0-P0.50-TL-EP2.6, symbol MerlynESC:EG6288_C55058511
- added U6: EFM8BB21F16G, easyeda2kicad:QFN-20_L3.0-W3.0-P0.50-BL-EP1.7_EFM8BB21F16G, symbol MerlynESC:EFM8BB21F16G-C-QFN20
- added U7: INA139NA, easyeda2kicad:SOT-23-5_L3.0-W1.7-P0.95-LS2.8-BR, symbol MerlynESC:INA139NA_3K
Connections:
- net +12V: now also C15.2, D4.2 (A), D5.2 (A), D6.2 (A), U5.4 (VCC)
- net +3.3V: now also C16.1, R33.1, U6.4 (VDD)
- net +BATT: now also Q3.5 (D), Q3.6 (D), Q3.7 (D), Q3.8 (D), Q3.9 (D), Q11.5 (D), Q11.6 (D), Q11.7 (D), Q11.8 (D), Q11.9 (D), Q7.5 (D), Q7.6 (D), Q7.7 (D), Q7.8 (D), Q7.9 (D), Q9.5 (D), Q9.6 (D), Q9.7 (D), Q9.8 (D), Q9.9 (D), R17.1, U7.4 (VIN-); no longer BT1.1 (+)
- net GND: now also Q4.1 (S), Q4.2 (S), Q4.3 (S), C15.1, C16.2, C20.1, C21.2, Q10.1 (S), Q10.2 (S), Q10.3 (S), Q12.1 (S), Q12.2 (S), Q12.3 (S), Q8.1 (S), Q8.2 (S), Q8.3 (S), R19.2, R24.2, R29.2, R34.1, U5.25 (EP), U5.6 (GND), U6.12 (GND), U6.21 (GND), U6.3 (GND), U7.2 (GND)
- new net: C20.2, R34.2, R35.2, U7.1 (OUT)
- new net: BT1.1 (+), C21.1, R17.2, U7.3 (VIN+), U7.5 (V+)
- new net: Q10.4 (G), R27.1
- new net: Q9.4 (G), R26.1
- new net: C18.1, U5.15 (VS2)
- new net: C18.2, D5.1 (K), U5.17 (VB2)
- new net: C17.1, U5.18 (VS1)
- new net: C17.2, D4.1 (K), U5.20 (VB1)
- new net: C19.1, U5.12 (VS3)
- new net: C19.2, D6.1 (K), U5.14 (VB3)
- new net: Q7.4 (G), R21.1
- new net: Q11.4 (G), R31.1
- new net: Q8.4 (G), R22.1
- new net: Q12.4 (G), R32.1
- new net CSense: R35.1
- new net M2_BEMF1: R18.2, R19.1, R20.1, U6.20 (P0.2)
- new net M2_BEMF2: R23.2, R24.1, R25.1, U6.2 (P0.0)
- new net M2_BEMF3: R28.2, R29.1, R30.1, U6.1 (P0.1)
- new net M2_BEMFCommon: R18.1, R23.1, R28.1, U6.19 (P0.3)
- new net M2_C2CK: R33.2, U6.5 (RSTB/C2CK)
- new net M2_C2D: U6.6 (P2.0/C2D)
- new net M2_DSHOT: U6.17 (P0.5)
- new net M2_H01: R21.2, U5.19 (HO1)
- new net M2_H02: R26.2, U5.16 (HO2)
- new net M2_H03: R31.2, U5.13 (HO3)
- new net M2_HIN1: U5.22 (HIN1), U6.14 (P1.0)
- new net M2_HIN2: U5.23 (HIN2), U6.11 (P1.2)
- new net M2_HIN3: U5.24 (HIN3), U6.9 (P1.4)
- new net M2_LIN1: U5.1 (LIN1), U6.13 (P1.1)
- new net M2_LIN2: U5.2 (LIN2), U6.10 (P1.3)
- new net M2_LIN3: U5.3 (LIN3), U6.8 (P1.5)
- new net M2_LO1: R22.2, U5.11 (LO1)
- new net M2_LO2: R27.2, U5.10 (LO2)
- new net M2_LO3: R32.2, U5.9 (LO3)
- new net M2_PHASE1: M2.1 (1/A/U), Q7.1 (S), Q7.2 (S), Q7.3 (S), Q8.5 (D), Q8.6 (D), Q8.7 (D), Q8.8 (D), Q8.9 (D), R20.2
- new net M2_PHASE2: M2.2 (2/B/V), Q10.5 (D), Q10.6 (D), Q10.7 (D), Q10.8 (D), Q10.9 (D), Q9.1 (S), Q9.2 (S), Q9.3 (S), R25.2
- new net M2_PHASE3: M2.3 (3/C/W), Q11.1 (S), Q11.2 (S), Q11.3 (S), Q12.5 (D), Q12.6 (D), Q12.7 (D), Q12.8 (D), Q12.9 (D), R30.2
- no-connect marks 8 -> 16
Other:
- note added: "Motor 2"
- moved on the sheet: BT1, C3, C4, C5, C6, C7, C8

Commit message: checkpoint
Parts:
- added C22, C23, C27, C28: 0.1uF, easyeda2kicad:C_0402_1005Metric, symbol Device:C_Small
- added C24, C25, C26, C29, C30, C31: 1uF, easyeda2kicad:C_0402_1005Metric, symbol Device:C_Small
- added D10, D11, D12, D7, D8, D9: T4, Diode_SMD:D_SOD-923, symbol Device:D_Small
- added H1, H4, H6, H8: C2CK, symbol MerlynESC:C2CK
- added H2, H5, H7, H9: C2D, symbol MerlynESC:C2D
- added H3: ESC Header, easyeda2kicad:ESC Header, symbol MerlynESC:ESC
- added M3, M4: BLDC Motor, easyeda2kicad:MotorPad, symbol MerlynESC:BLDC Motor
- added Q13, Q14, Q15, Q16, Q17, Q18, Q19, Q20, Q21, Q22, Q23, Q24: JMSL0302AU, easyeda2kicad:DFN-8_L3.2-W3.1-P0.65-LS3.4-BL, symbol MerlynESC:JMSL0302AU
- added R36, R41, R46, R52, R57, R62: 4.7k, easyeda2kicad:R_0402_1005Metric, symbol Device:R_Small
- added R37, R42, R47, R51, R53, R58, R63, R67: 1k, easyeda2kicad:R_0402_1005Metric, symbol Device:R_Small
- added R38, R43, R48, R54, R59, R64: 10k, easyeda2kicad:R_0402_1005Metric, symbol Device:R_Small
- added R39, R40, R44, R45, R49, R50, R55, R56, R60, R61, R65, R66: 10, easyeda2kicad:R_0402_1005Metric, symbol Device:R_Small
- added U10, U8: EG6288, easyeda2kicad:QFN-24_L4.0-W4.0-P0.50-TL-EP2.6, symbol MerlynESC:EG6288_C55058511
- added U11, U9: EFM8BB21F16G, easyeda2kicad:QFN-20_L3.0-W3.0-P0.50-BL-EP1.7_EFM8BB21F16G, symbol MerlynESC:EFM8BB21F16G-C-QFN20
- BT1: footprint (none) -> easyeda2kicad:PowerPad
- C10, C11, C12, C13, C14, C15, C16, C17, C18, C19, C20, C21: footprint Capacitor_SMD:C_0402_1005Metric -> easyeda2kicad:C_0402_1005Metric
- M1, M2: footprint (none) -> easyeda2kicad:MotorPad
- R1, R10, R11, R12, R13, R14, R15, R16, R18, R19, R2, R20, R21, R22, R23, R24, R25, R26, R27, R28, R29, R3, R30, R31, R32, R33, R34, R35, R4, R5, R6, R7, R8, R9: footprint Resistor_SMD:R_0402_1005Metric -> easyeda2kicad:R_0402_1005Metric
Connections:
- net +12V: now also C22.2, C27.2, D10.2 (A), D11.2 (A), D12.2 (A), D7.2 (A), D8.2 (A), D9.2 (A), U10.4 (VCC), U8.4 (VCC)
- net +3.3V: now also C23.1, C28.1, R51.1, R67.1, U11.4 (VDD), U9.4 (VDD)
- net +BATT: now also H3.8 (BAT+), Q13.5 (D), Q13.6 (D), Q13.7 (D), Q13.8 (D), Q13.9 (D), Q15.5 (D), Q15.6 (D), Q15.7 (D), Q15.8 (D), Q15.9 (D), Q17.5 (D), Q17.6 (D), Q17.7 (D), Q17.8 (D), Q17.9 (D), Q19.5 (D), Q19.6 (D), Q19.7 (D), Q19.8 (D), Q19.9 (D), Q21.5 (D), Q21.6 (D), Q21.7 (D), Q21.8 (D), Q21.9 (D), Q23.5 (D), Q23.6 (D), Q23.7 (D), Q23.8 (D), Q23.9 (D)
- net CSense: now also H3.5 (CUR)
- net GND: now also C22.1, C23.2, C27.1, C28.2, H3.7 (GND), Q14.1 (S), Q14.2 (S), Q14.3 (S), Q16.1 (S), Q16.2 (S), Q16.3 (S), Q18.1 (S), Q18.2 (S), Q18.3 (S), Q20.1 (S), Q20.2 (S), Q20.3 (S), Q22.1 (S), Q22.2 (S), Q22.3 (S), Q24.1 (S), Q24.2 (S), Q24.3 (S), R37.2, R42.2, R47.2, R53.2, R58.2, R63.2, U10.25 (EP), U10.6 (GND), U11.12 (GND), U11.21 (GND), U11.3 (GND), U8.25 (EP), U8.6 (GND), U9.12 (GND), U9.21 (GND), U9.3 (GND)
- net M1_C2CK: now also H1.1 (C2CK)
- net M1_C2D: now also H2.1 (C2D)
- net M1_DSHOT: now also H3.4 (M1)
- net M2_C2CK: now also H4.1 (C2CK)
- net M2_C2D: now also H5.1 (C2D)
- net M2_DSHOT: now also H3.3 (M2)
- new net: C29.2, D10.1 (K), U10.20 (VB1)
- new net: Q19.4 (G), R55.1
- new net: C24.1, U8.18 (VS1)
- new net: C24.2, D7.1 (K), U8.20 (VB1)
- new net: Q13.4 (G), R39.1
- new net: Q24.4 (G), R66.1
- new net: Q22.4 (G), R61.1
- new net: C26.1, U8.12 (VS3)
- new net: C26.2, D9.1 (K), U8.14 (VB3)
- new net: C25.1, U8.15 (VS2)
- new net: C25.2, D8.1 (K), U8.17 (VB2)
- new net: C31.2, D12.1 (K), U10.14 (VB3)
- new net: Q20.4 (G), R56.1
- new net: Q17.4 (G), R49.1
- new net: C30.2, D11.1 (K), U10.17 (VB2)
- new net: Q15.4 (G), R44.1
- new net: C31.1, U10.12 (VS3)
- new net: Q21.4 (G), R60.1
- new net: Q18.4 (G), R50.1
- new net: Q23.4 (G), R65.1
- new net: Q14.4 (G), R40.1
- new net: C30.1, U10.15 (VS2)
- new net: C29.1, U10.18 (VS1)
- new net: Q16.4 (G), R45.1
- new net M3_BEMF1: R36.2, R37.1, R38.1, U9.20 (P0.2)
- new net M3_BEMF2: R41.2, R42.1, R43.1, U9.2 (P0.0)
- new net M3_BEMF3: R46.2, R47.1, R48.1, U9.1 (P0.1)
- new net M3_BEMFCommon: R36.1, R41.1, R46.1, U9.19 (P0.3)
- new net M3_C2CK: H6.1 (C2CK), R51.2, U9.5 (RSTB/C2CK)
- new net M3_C2D: H7.1 (C2D), U9.6 (P2.0/C2D)
- new net M3_DSHOT: H3.2 (M3), U9.17 (P0.5)
- new net M3_H01: R39.2, U8.19 (HO1)
- new net M3_H02: R44.2, U8.16 (HO2)
- new net M3_H03: R49.2, U8.13 (HO3)
- new net M3_HIN1: U8.22 (HIN1), U9.14 (P1.0)
- new net M3_HIN2: U8.23 (HIN2), U9.11 (P1.2)
- new net M3_HIN3: U8.24 (HIN3), U9.9 (P1.4)
- new net M3_LIN1: U8.1 (LIN1), U9.13 (P1.1)
- new net M3_LIN2: U8.2 (LIN2), U9.10 (P1.3)
- new net M3_LIN3: U8.3 (LIN3), U9.8 (P1.5)
- new net M3_LO1: R40.2, U8.11 (LO1)
- new net M3_LO2: R45.2, U8.10 (LO2)
- new net M3_LO3: R50.2, U8.9 (LO3)
- new net M3_PHASE1: M3.1 (1/A/U), Q13.1 (S), Q13.2 (S), Q13.3 (S), Q14.5 (D), Q14.6 (D), Q14.7 (D), Q14.8 (D), Q14.9 (D), R38.2
- new net M3_PHASE2: M3.2 (2/B/V), Q15.1 (S), Q15.2 (S), Q15.3 (S), Q16.5 (D), Q16.6 (D), Q16.7 (D), Q16.8 (D), Q16.9 (D), R43.2
- new net M3_PHASE3: M3.3 (3/C/W), Q17.1 (S), Q17.2 (S), Q17.3 (S), Q18.5 (D), Q18.6 (D), Q18.7 (D), Q18.8 (D), Q18.9 (D), R48.2
- new net M4_BEMF1: R52.2, R53.1, R54.1, U11.20 (P0.2)
- new net M4_BEMF2: R57.2, R58.1, R59.1, U11.2 (P0.0)
- new net M4_BEMF3: R62.2, R63.1, R64.1, U11.1 (P0.1)
- new net M4_BEMFCommon: R52.1, R57.1, R62.1, U11.19 (P0.3)
- new net M4_C2CK: H8.1 (C2CK), R67.2, U11.5 (RSTB/C2CK)
- new net M4_C2D: H9.1 (C2D), U11.6 (P2.0/C2D)
- new net M4_DSHOT: H3.1 (M4), U11.17 (P0.5)
- new net M4_H01: R55.2, U10.19 (HO1)
- new net M4_H02: R60.2, U10.16 (HO2)
- new net M4_H03: R65.2, U10.13 (HO3)
- new net M4_HIN1: U10.22 (HIN1), U11.14 (P1.0)
- new net M4_HIN2: U10.23 (HIN2), U11.11 (P1.2)
- new net M4_HIN3: U10.24 (HIN3), U11.9 (P1.4)
- new net M4_LIN1: U10.1 (LIN1), U11.13 (P1.1)
- new net M4_LIN2: U10.2 (LIN2), U11.10 (P1.3)
- new net M4_LIN3: U10.3 (LIN3), U11.8 (P1.5)
- new net M4_LO1: R56.2, U10.11 (LO1)
- new net M4_LO2: R61.2, U10.10 (LO2)
- new net M4_LO3: R66.2, U10.9 (LO3)
- new net M4_PHASE1: M4.1 (1/A/U), Q19.1 (S), Q19.2 (S), Q19.3 (S), Q20.5 (D), Q20.6 (D), Q20.7 (D), Q20.8 (D), Q20.9 (D), R54.2
- new net M4_PHASE2: M4.2 (2/B/V), Q21.1 (S), Q21.2 (S), Q21.3 (S), Q22.5 (D), Q22.6 (D), Q22.7 (D), Q22.8 (D), Q22.9 (D), R59.2
- new net M4_PHASE3: M4.3 (3/C/W), Q23.1 (S), Q23.2 (S), Q23.3 (S), Q24.5 (D), Q24.6 (D), Q24.7 (D), Q24.8 (D), Q24.9 (D), R64.2
- no-connect marks 16 -> 33
Other:
- note added: "Motor 3"
- note added: "Motor 4"
- moved on the sheet: BT1, C1, C10, C11, C12, C13, C14, C15, C16, C17, C18, C19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

Commit message: checkpoint
Connections:
- net M1_BEMF1: now also U3.1 (P0.1); no longer U3.20 (P0.2)
- net M1_BEMF2: now also U3.20 (P0.2); no longer U3.2 (P0.0)
- net M1_BEMF3: now also U3.19 (P0.3); no longer U3.1 (P0.1)
- net M1_BEMFCommon: now also U3.2 (P0.0); no longer U3.19 (P0.3)
- net M2_BEMF1: now also U6.1 (P0.1); no longer U6.20 (P0.2)
- net M2_BEMF2: now also U6.20 (P0.2); no longer U6.2 (P0.0)
- net M2_BEMF3: now also U6.19 (P0.3); no longer U6.1 (P0.1)
- net M2_BEMFCommon: now also U6.2 (P0.0); no longer U6.19 (P0.3)
- net M3_BEMF1: now also U9.1 (P0.1); no longer U9.20 (P0.2)
- net M3_BEMF2: now also U9.20 (P0.2); no longer U9.2 (P0.0)
- net M3_BEMF3: now also U9.19 (P0.3); no longer U9.1 (P0.1)
- net M3_BEMFCommon: now also U9.2 (P0.0); no longer U9.19 (P0.3)
- net M4_BEMF1: now also U11.1 (P0.1); no longer U11.20 (P0.2)
- net M4_BEMF2: now also U11.20 (P0.2); no longer U11.2 (P0.0)
- net M4_BEMF3: now also U11.19 (P0.3); no longer U11.1 (P0.1)
- net M4_BEMFCommon: now also U11.2 (P0.0); no longer U11.19 (P0.3)
Changed lines of the file:
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@@
 	(global_label "M1_BEMF3"
 		(shape input)
-		(at 308.61 129.54 90)
+		(at 323.85 147.32 0)
 		(fields_autoplaced yes)
 		(effects
@@
 		)
 		(property "Intersheetrefs" "${INTERSHEET_REFS}"
-			(at 308.61 116.7578 90)
+			(at 343.5263 147.32 0)
 			(effects
 				(font
@@
 	(global_label "M2_BEMFCommon"
 		(shape input)
-		(at 544.83 147.32 0)
+		(at 527.05 129.54 90)
 		(fields_autoplaced yes)
 		(effects
@@
 		)
 		(property "Intersheetrefs" "${INTERSHEET_REFS}"
-			(at 564.5063 147.32 0)
+			(at 527.05 116.7578 90)
 			(effects
 				(font
@@
 	(global_label "M1_BEMF1"
 		(shape input)
-		(at 323.85 144.78 0)
+		(at 308.61 129.54 90)
 		(fields_autoplaced yes)
 		(effects
@@
 		)
 		(property "Intersheetrefs" "${INTERSHEET_REFS}"
-			(at 336.6322 144.78 0)
+			(at 308.61 116.7578 90)
 			(effects
 				(font
@@
 	(global_label "M2_BEMF1"
 		(shape input)
-		(at 544.83 144.78 0)
+		(at 529.59 129.54 90)
 		(fields_autoplaced yes)
 		(effects
@@
 		)
 		(property "Intersheetrefs" "${INTERSHEET_REFS}"
-			(at 557.6122 144.78 0)
+			(at 529.59 116.7578 90)
 			(effects
 				(font
@@
 	(global_label "M3_BEMF3"
 		(shape input)
-		(at 308.61 299.72 90)
+		(at 323.85 317.5 0)
 		(fields_autoplaced yes)
 		(effects
@@
 		)
 		(property "Intersheetrefs" "${INTERSHEET_REFS}"
-			(at 308.61 286.9378 90)
+			(at 343.5263 317.5 0)
 			(effects
 				(font
@@
 	(global_label "M4_BEMF2"
 		(shape input)
-		(at 527.05 299.72 90)
+		(at 544.83 314.96 0)
 		(fields_autoplaced yes)
 		(effects
@@
 		)
 		(property "Intersheetrefs" "${INTERSHEET_REFS}"
-			(at 527.05 286.9378 90)
+			(at 557.6122 314.96 0)
 			(effects
 				(font
@@
 	(global_label "M1_BEMFCommon"
 		(shape input)
-		(at 323.85 147.32 0)
+		(at 306.07 129.54 90)
 		(fields_autoplaced yes)
 		(effects
@@
 		)
 		(property "Intersheetrefs" "${INTERSHEET_REFS}"
-			(at 343.5263 147.32 0)
+			(at 306.07 116.7578 90)
 			(effects
 				(font
@@
 	(global_label "M1_BEMF2"
 		(shape input)
-		(at 306.07 129.54 90)
+		(at 323.85 144.78 0)
 		(fields_autoplaced yes)
 		(effects
@@
 		)
 		(property "Intersheetrefs" "${INTERSHEET_REFS}"
-			(at 306.07 116.7578 90)
+			(at 336.6322 144.78 0)
 			(effects
 				(font
@@
 	(global_label "M4_BEMFCommon"
 		(shape input)
-		(at 544.83 317.5 0)
+		(at 527.05 299.72 90)
 		(fields_autoplaced yes)
 		(effects
@@
 		)
 		(property "Intersheetrefs" "${INTERSHEET_REFS}"
-			(at 564.5063 317.5 0)
+			(at 527.05 286.9378 90)
 			(effects
 				(font
@@
 	(global_label "M3_BEMF1"
 		(shape input)
-		(at 323.85 314.96 0)
+		(at 308.61 299.72 90)
 		(fields_autoplaced yes)
 		(effects
@@
 		)
 		(property "Intersheetrefs" "${INTERSHEET_REFS}"
-			(at 336.6322 314.96 0)
+			(at 308.61 286.9378 90)
 			(effects
 				(font
@@
 	(global_label "M3_BEMFCommon"
 		(shape input)
-		(at 323.85 317.5 0)
+		(at 306.07 299.72 90)
 		(fields_autoplaced yes)
 		(effects
@@
 		)
 		(property "Intersheetrefs" "${INTERSHEET_REFS}"
-			(at 343.5263 317.5 0)
+			(at 306.07 286.9378 90)
 			(effects
 				(font
@@
 	(global_label "M2_BEMF3"
 		(shape input)
-		(at 529.59 129.54 90)
+		(at 544.83 147.32 0)
 		(fields_autoplaced yes)
 		(effects
@@
 		)
 		(property "Intersheetrefs" "${INTERSHEET_REFS}"
-			(at 529.59 116.7578 90)
+			(at 564.5063 147.32 0)
 			(effects
 				(font
@@
 	(global_label "M4_BEMF3"
 		(shape input)
-		(at 529.59 299.72 90)
+		(at 544.83 317.5 0)
 		(fields_autoplaced yes)
 		(effects
@@
 		)
 		(property "Intersheetrefs" "${INTERSHEET_REFS}"
-			(at 529.59 286.9378 90)
+			(at 564.5063 317.5 0)
 			(effects
 				(font
@@
 	(global_label "M2_BEMF2"
 		(shape input)
-		(at 527.05 129.54 90)
+		(at 544.83 144.78 0)
 		(fields_autoplaced yes)
 		(effects
@@
 		)
 		(property "Intersheetrefs" "${INTERSHEET_REFS}"
-			(at 527.05 116.7578 90)
+			(at 557.6122 144.78 0)
 			(effects
 				(font
@@
 	(global_label "M3_BEMF2"
 		(shape input)
-		(at 306.07 299.72 90)
+		(at 323.85 314.96 0)
 		(fields_autoplaced yes)
 		(effects
@@
 		)
 		(property "Intersheetrefs" "${INTERSHEET_REFS}"
-			(at 306.07 286.9378 90)
+			(at 336.6322 314.96 0)
 			(effects
 				(font
@@
 	(global_label "M4_BEMF1"
 		(shape input)
-		(at 544.83 314.96 0)
+		(at 529.59 299.72 90)
 		(fields_autoplaced yes)
 		(effects
@@
 		)
 		(property "Intersheetrefs" "${INTERSHEET_REFS}"
-			(at 557.6122 314.96 0)
+			(at 529.59 286.9378 90)
 			(effects
 				(font

Commit message: checkpoint
Parts:
- H1, H2, H4, H5, H6, H7, H8, H9: footprint (none) -> easyeda2kicad:TestPoint
Changed lines of the file:
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@@
 			)
 		)
-		(property "Footprint" ""
+		(property "Footprint" "easyeda2kicad:TestPoint"
 			(at 147.32 337.82 0)
 			(effects
@@
 			)
 		)
-		(property "Footprint" ""
+		(property "Footprint" "easyeda2kicad:TestPoint"
 			(at 378.46 167.64 0)
 			(effects
@@
 			)
 		)
-		(property "Footprint" ""
+		(property "Footprint" "easyeda2kicad:TestPoint"
 			(at 368.3 337.82 0)
 			(effects
@@
 			)
 		)
-		(property "Footprint" ""
+		(property "Footprint" "easyeda2kicad:TestPoint"
 			(at 157.48 167.64 0)
 			(effects
@@
 			)
 		)
-		(property "Footprint" ""
+		(property "Footprint" "easyeda2kicad:TestPoint"
 			(at 147.32 167.64 0)
 			(effects
@@
 			)
 		)
-		(property "Footprint" ""
+		(property "Footprint" "easyeda2kicad:TestPoint"
 			(at 157.48 337.82 0)
 			(effects
@@
 			)
 		)
-		(property "Footprint" ""
+		(property "Footprint" "easyeda2kicad:TestPoint"
 			(at 378.46 337.82 0)
 			(effects
@@
 			)
 		)
-		(property "Footprint" ""
+		(property "Footprint" "easyeda2kicad:TestPoint"
 			(at 368.3 167.64 0)
 			(effects
