File: PCB/ESC/MerlynESC.kicad_sch (KiCad schematic)
At the start: 159 parts, among them M1 BLDC Motor, M2 BLDC Motor, M3 BLDC Motor, M4 BLDC Motor, Q1 JMSL0302AU, Q10 JMSL0302AU, Q11 JMSL0302AU, Q12 JMSL0302AU, Q13 JMSL0302AU, Q14 JMSL0302AU, Q15 JMSL0302AU, Q16 JMSL0302AU, Q17 JMSL0302AU, Q18 JMSL0302AU, Q19 JMSL0302AU, Q2 JMSL0302AU, Q20 JMSL0302AU, Q21 JMSL0302AU, Q22 JMSL0302AU, Q23 JMSL0302AU, Q24 JMSL0302AU, Q3 JMSL0302AU, Q4 JMSL0302AU, Q5 JMSL0302AU, Q6 JMSL0302AU, Q7 JMSL0302AU, Q8 JMSL0302AU, Q9 JMSL0302AU, U1 HT75C0-1, U10 EG6288, U11 EFM8BB21F16G, U2 HT7533-1, U3 EFM8BB21F16G, U4 EG6288, U5 EG6288, U6 EFM8BB21F16G, U7 INA139NA, U8 EG6288, U9 EFM8BB21F16G

Commit message: checkpoint
Parts:
- BT1, H1, H2, H4, H5, H6, H7, H8, H9, M1, M2, M3, M4: now left out of the parts list
- C1: footprint Capacitor_SMD:C_0805_2012Metric -> easyeda2kicad:C_0805_2012Metric
- C2, C9: footprint Capacitor_SMD:C_0603_1608Metric -> easyeda2kicad:C_0603_1608Metric
- C3, C4, C5, C6, C7, C8: footprint Capacitor_SMD:C_1206_3216Metric -> easyeda2kicad:C_1206_3216Metric
- D1, D10, D11, D12, D2, D3, D4, D5, D6, D7, D8, D9: footprint Diode_SMD:D_SOD-923 -> easyeda2kicad:D_SOD-923
Changed lines of the file:
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@@
 			)
 		)
-		(property "Footprint" "Diode_SMD:D_SOD-923"
+		(property "Footprint" "easyeda2kicad:D_SOD-923"
 			(at 553.72 234.95 90)
 			(effects
@@
 			)
 		)
-		(property "Footprint" "Diode_SMD:D_SOD-923"
+		(property "Footprint" "easyeda2kicad:D_SOD-923"
 			(at 332.74 64.77 90)
 			(effects
@@
 			)
 		)
-		(property "Footprint" "Diode_SMD:D_SOD-923"
+		(property "Footprint" "easyeda2kicad:D_SOD-923"
 			(at 332.74 242.57 90)
 			(effects
@@
 			)
 		)
-		(property "Footprint" "Capacitor_SMD:C_0603_1608Metric"
+		(property "Footprint" "easyeda2kicad:C_0603_1608Metric"
 			(at 118.11 68.58 0)
 			(effects
@@
 		(unit 1)
 		(exclude_from_sim no)
-		(in_bom yes)
+		(in_bom no)
 		(on_board yes)
 		(dnp no)
@@
 			)
 		)
-		(property "Footprint" "Diode_SMD:D_SOD-923"
+		(property "Footprint" "easyeda2kicad:D_SOD-923"
 			(at 553.72 250.19 90)
 			(effects
@@
 			)
 		)
-		(property "Footprint" "Diode_SMD:D_SOD-923"
+		(property "Footprint" "easyeda2kicad:D_SOD-923"
 			(at 332.74 72.39 90)
 			(effects
@@
 			)
 		)
-		(property "Footprint" "Diode_SMD:D_SOD-923"
+		(property "Footprint" "easyeda2kicad:D_SOD-923"
 			(at 332.74 80.01 90)
 			(effects
@@
 			)
 		)
-		(property "Footprint" "Diode_SMD:D_SOD-923"
+		(property "Footprint" "easyeda2kicad:D_SOD-923"
 			(at 553.72 80.01 90)
 			(effects
@@
 			)
 		)
-		(property "Footprint" "Diode_SMD:D_SOD-923"
+		(property "Footprint" "easyeda2kicad:D_SOD-923"
 			(at 332.74 234.95 90)
 			(effects
@@
 			)
 		)
-		(property "Footprint" "Diode_SMD:D_SOD-923"
+		(property "Footprint" "easyeda2kicad:D_SOD-923"
 			(at 553.72 242.57 90)
 			(effects
@@
 			)
 		)
-		(property "Footprint" "Capacitor_SMD:C_1206_3216Metric"
+		(property "Footprint" "easyeda2kicad:C_1206_3216Metric"
 			(at 111.76 167.64 0)
 			(effects
@@
 			)
 		)
-		(property "Footprint" "Diode_SMD:D_SOD-923"
+		(property "Footprint" "easyeda2kicad:D_SOD-923"
 			(at 553.72 64.77 90)
 			(effects
@@
 			)
 		)
-		(property "Footprint" "Diode_SMD:D_SOD-923"
+		(property "Footprint" "easyeda2kicad:D_SOD-923"
 			(at 332.74 250.19 90)
 			(effects
@@
 		(unit 1)
 		(exclude_from_sim no)
-		(in_bom yes)
+		(in_bom no)
 		(on_board yes)
 		(dnp no)
@@
 		(unit 1)
 		(exclude_from_sim no)
-		(in_bom yes)
+		(in_bom no)
 		(on_board yes)
 		(dnp no)
@@
 			)
 		)
-		(property "Footprint" "Capacitor_SMD:C_1206_3216Metric"
+		(property "Footprint" "easyeda2kicad:C_1206_3216Metric"
 			(at 88.9 167.64 0)
 			(effects
@@
 		(unit 1)
 		(exclude_from_sim no)
-		(in_bom yes)
+		(in_bom no)
 		(on_board yes)
 		(dnp no)
@@
 		(unit 1)
 		(exclude_from_sim no)
-		(in_bom yes)
+		(in_bom no)
 		(on_board yes)
 		(dnp no)
@@
 		(unit 1)
 		(exclude_from_sim no)
-		(in_bom yes)
+		(in_bom no)
 		(on_board yes)
 		(dnp no)
@@
 			)
 		)
-		(property "Footprint" "Capacitor_SMD:C_1206_3216Metric"
+		(property "Footprint" "easyeda2kicad:C_1206_3216Metric"
 			(at 81.28 167.64 0)
 			(effects
@@
 			)
 		)
-		(property "Footprint" "Capacitor_SMD:C_0603_1608Metric"
+		(property "Footprint" "easyeda2kicad:C_0603_1608Metric"
 			(at 114.3 39.37 0)
 			(effects
@@
 			)
 		)
-		(property "Footprint" "Capacitor_SMD:C_0805_2012Metric"
+		(property "Footprint" "easyeda2kicad:C_0805_2012Metric"
 			(at 99.06 68.58 0)
 			(effects
@@
 			)
 		)
-		(property "Footprint" "Capacitor_SMD:C_1206_3216Metric"
+		(property "Footprint" "easyeda2kicad:C_1206_3216Metric"
 			(at 73.66 167.64 0)
 			(effects
@@
 			)
 		)
-		(property "Footprint" "Capacitor_SMD:C_1206_3216Metric"
+		(property "Footprint" "easyeda2kicad:C_1206_3216Metric"
 			(at 104.14 167.64 0)
 			(effects
@@
 			)
 		)
-		(property "Footprint" "Diode_SMD:D_SOD-923"
+		(property "Footprint" "easyeda2kicad:D_SOD-923"
 			(at 553.72 72.39 90)
 			(effects
@@
 		(unit 1)
 		(exclude_from_sim no)
-		(in_bom yes)
+		(in_bom no)
 		(on_board yes)
 		(dnp no)
@@
 		(unit 1)
 		(exclude_from_sim no)
-		(in_bom yes)
+		(in_bom no)
 		(on_board yes)
 		(dnp no)
@@
 		(unit 1)
 		(exclude_from_sim no)
-		(in_bom yes)
+		(in_bom no)
 		(on_board yes)
 		(dnp no)
@@
 		(unit 1)
 		(exclude_from_sim no)
-		(in_bom yes)
+		(in_bom no)
 		(on_board yes)
 		(dnp no)
@@
 		(unit 1)
 		(exclude_from_sim no)
-		(in_bom yes)
+		(in_bom no)
 		(on_board yes)
 		(dnp no)
@@
 			)
 		)
-		(property "Footprint" "Capacitor_SMD:C_1206_3216Metric"
+		(property "Footprint" "easyeda2kicad:C_1206_3216Metric"
 			(at 96.52 167.64 0)
 			(effects
@@
 		(unit 1)
 		(exclude_from_sim no)
-		(in_bom yes)
+		(in_bom no)
 		(on_board yes)
 		(dnp no)
@@
 		(unit 1)
 		(exclude_from_sim no)
-		(in_bom yes)
+		(in_bom no)
 		(on_board yes)
 		(dnp no)

Commit message: checkpoint
Other:
- note added: "12v Reg"
- note added: "3.3v Reg"
- note added: "Bulk Capacitor"
- note added: "Connector"
- note added: "Current Sense"
- note added: "Power Regulation"
- moved on the sheet: BT1, C1, C2, C20, C21, C3, C4, C5, C6, C7, C8, C9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

Commit message: ESC Rev 2. Connected gate driver VS pin to motor phase
Connections:
- net M1_PHASE1: now also C11.1, U4.18 (VS1)
- net M1_PHASE2: now also C12.1, U4.15 (VS2)
- net M1_PHASE3: now also C13.1, U4.12 (VS3)
- net M2_PHASE1: now also C17.1, U5.18 (VS1)
- net M2_PHASE2: now also C18.1, U5.15 (VS2)
- net M2_PHASE3: now also C19.1, U5.12 (VS3)
- net M3_PHASE1: now also C24.1, U8.18 (VS1)
- net M3_PHASE2: now also C25.1, U8.15 (VS2)
- net M3_PHASE3: now also C26.1, U8.12 (VS3)
- net M4_PHASE1: now also C29.1, U10.18 (VS1)
- net M4_PHASE2: now also C30.1, U10.15 (VS2)
- net M4_PHASE3: now also C31.1, U10.12 (VS3)
